File: MiniSNH v1.0/Fabrication/MiniSNH v1.0 - Main.kicad_pcb (KiCad board)
At the start: 2 copper layers, 45 x 128.5 mm, 86 parts, among them J2 IDC_2x05, Q1 BC548, Q2 BC549, Q3 MMBFJ113, U1 TL072, U2 TL072, U3 TL072, U4 4081, U5 TL072, U6 TL072

Commit message: Added v1.1
Parts:
- removed ? (x9): , Wire_Pads:SolderWirePad_single_0-8mmDrill
- removed G*** (x2): LOGO, LOGO
Other:
- board size 45 x 128.5 mm -> 20 x 107.9 mm
