File: MiniSNH v1.1/MiniSNH.kicad_pcb (KiCad board)
At the start: 2 copper layers, 45 x 128.5 mm, 86 parts, among them J2 IDC_2x05, Q1 BC548, Q2 BC549, Q3 MMBFJ113, U1 TL072, U2 TL072, U3 TL072, U4 4081, U5 TL072, U6 TL072

Commit message: Added v1.1
Parts:
- added C16: 100nF, Capacitor_SMD:C_0603_1608Metric_Pad1.08x0.95mm_HandSolder, B.Cu at (144.3, 101.6)
- added C19: 100nF, Capacitor_SMD:C_0603_1608Metric_Pad1.08x0.95mm_HandSolder, B.Cu at (152.9, 106.1)
- added R30: 10k, Resistor_SMD:R_0603_1608Metric_Pad0.98x0.95mm_HandSolder, B.Cu at (139.8, 149.5)
- added R31: 10k, Resistor_SMD:R_0603_1608Metric_Pad0.98x0.95mm_HandSolder, B.Cu at (141.4, 149.5)
- added REF**: Panel_4HP, benjiaomodular:Panel_4HP, F.Cu at (110.0, 49.0)
- Q1: value BC548 -> BC549
- moved R21 18.8 mm to (136.0, 149.1), turned to 90 degrees
- moved R18 17.7 mm to (152.6, 149.1), turned to 90 degrees
- moved R19 15.4 mm to (151.0, 149.1), turned to -90 degrees
- moved D2 15.1 mm to (152.6, 146.0)
- moved D3 15.0 mm to (137.5, 146.0)
- moved R22 11.1 mm to (139.5, 160.7), turned to 180 degrees
- moved R15 11.0 mm to (150.5, 162.1), turned to 180 degrees
- moved R17 11.0 mm to (139.5, 162.3), turned to 0 degrees
- moved C18 10.5 mm to (146.5, 71.3), turned to 180 degrees
- moved GATE_OUT2 10.1 mm to (140.0, 167.9)
- moved GATE_OUT1 10.0 mm to (150.0, 167.9)
- moved C17 9.32 mm to (139.0, 65.9)
- moved R14 8.58 mm to (150.5, 160.5)
- moved C4 7.69 mm to (145.8, 96.2), turned to -90 degrees
- moved R7 7.20 mm to (144.2, 96.2), turned to -90 degrees
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Connections:
- C7 pad 1: Net-(C7-Pad1) -> GATE_IN
- GATE_IN1 pad T: Net-(C7-Pad1) -> GATE_IN
- GATE_IN1 pad TN: GATE_IN -> unconnected-(GATE_IN1-PadTN)
- PROB_IN1 pad TN: Net-(PROBABILITY1-Pad2) -> Net-(PROB_IN1-PadTN)
- U3 pad 1: Net-(D3-Pad2) -> Net-(D2-Pad2)
- U3 pad 2: Net-(D3-Pad2) -> Net-(D2-Pad2)
- U3 pad 3: Net-(R16-Pad2) -> Net-(R14-Pad2)
- U3 pad 5: Net-(R14-Pad2) -> Net-(R16-Pad2)
- U3 pad 6: Net-(D2-Pad2) -> Net-(D3-Pad2)
- U3 pad 7: Net-(D2-Pad2) -> Net-(D3-Pad2)
- U5 pad 4: +12V -> -12V
- U5 pad 8: -12V -> +12V
- U6 pad 4: +12V -> -12V
- U6 pad 8: -12V -> +12V
Routing:
- net +12V: track 197.4 -> 171.5 mm, vias 9 -> 8
- net Net-(D2-Pad1): track 17.1 -> 2.17 mm
- net -12V: track 156.1 -> 141.6 mm, vias 7 -> 5
- net Net-(D3-Pad1): track 17.3 -> 2.80 mm
- net Net-(R7-Pad1): track 9.85 -> 18.7 mm
- net GATE_IN: track 46.1 -> 54.5 mm
- net Net-(PROB_IN1-PadTN): track 0.00 -> 6.54 mm
- net Net-(Q3-Pad1): track 5.34 -> 10.2 mm
- net GATE_OUT1: track 3.46 -> 6.93 mm
- net Net-(D5-Pad2): track 9.68 -> 13.1 mm
- net Net-(Q2-Pad1): track 19.1 -> 21.7 mm
- net Net-(D2-Pad2): track 21.9 -> 19.4 mm
- net Net-(R16-Pad2): track 7.40 -> 9.66 mm
- net Net-(PROBABILITY1-Pad2): track 13.7 -> 11.7 mm, vias 0 -> 1
- net Net-(R14-Pad1): track 32.8 -> 30.9 mm, vias 0 -> 2
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Other:
- board text added: "MiniSNH v1.1"
- board text added: "benjiaomodular"
