File: MiniSNH v1.1/MiniSNH.kicad_sch (KiCad schematic)
At the start: 70 parts, among them Q1 BC548, Q2 BC549, Q3 MMBFJ113, U1 TL072, U2 TL072, U3 TL072, U4 4081, U5 TL072, U6 TL072

Commit message: Added v1.1
Parts:
- added C16, C19: 100nF, Capacitor_SMD:C_0603_1608Metric_Pad1.08x0.95mm_HandSolder, symbol Device:C
- added R30, R31: 10k, Resistor_SMD:R_0603_1608Metric_Pad0.98x0.95mm_HandSolder, symbol Device:R
- Q1: value BC548 -> BC549
Connections:
- net +12V: now also U5.8 (V+), U6.8 (V+), C16.2; no longer U5.4 (V-), U6.4 (V-)
- net -12V: now also U5.4 (V-), U6.4 (V-), C19.1; no longer U5.8 (V+), U6.8 (V+)
- net GATE_IN: now also C7.1, GATE_IN1.T; no longer GATE_IN1.TN
- net GND: now also C16.1, C19.2, R31.2
- net at R16.2, R17.2: now also U3.5 (+); no longer U3.3 (+)
- net at D3.2 (A), R22.1: now also U3.6 (-), U3.7; no longer U3.1, U3.2 (-)
- net at R14.2, R15.2: now also U3.3 (+); no longer U3.5 (+)
- net at PROB_IN1.TN: now also R30.1, R31.1; no longer PROBABILITY1.2
- net at D2.2 (A), R19.1: now also U3.1, U3.2 (-); no longer U3.6 (-), U3.7
- new net: PROBABILITY1.2, R30.2
- no-connect marks 8 -> 9
Other:
- note added: "U1"
- note added: "U2"
- note added: "U3"
- note added: "U5"
- note added: "U6"
- title: (none) -> MiniSNH
- moved on the sheet: C15, C17, C18, D1, D2, D3, GATE_OUT1, GATE_OUT2, PROBABILITY1, PROB_IN1, Q2, R10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

Commit message: Added gerber files for v1.1
Other:
- note added: "Noise Source"
- note added: "Probability"
- note added: "SNH"
- moved on the sheet: C15
Changed lines of the file:
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@@
     (stroke (width 0) (type default) (color 0 0 0 0))
   )
-  (wire (pts (xy 176.276 176.784) (xy 176.276 191.77))
+  (wire (pts (xy 173.482 176.784) (xy 173.482 191.77))
     (stroke (width 0) (type default) (color 0 0 0 0))
   )
@@
     (stroke (width 0) (type default) (color 0 0 0 0))
   )
-  (wire (pts (xy 176.276 191.77) (xy 162.052 191.77))
+  (wire (pts (xy 173.482 191.77) (xy 162.052 191.77))
     (stroke (width 0) (type default) (color 0 0 0 0))
   )
@@
     (stroke (width 0) (type default) (color 0 0 0 0))
   )
-  (wire (pts (xy 162.052 164.338) (xy 176.276 164.338))
+  (wire (pts (xy 162.052 164.338) (xy 173.482 164.338))
     (stroke (width 0) (type default) (color 0 0 0 0))
   )
@@
     (stroke (width 0) (type default) (color 0 0 0 0))
   )
-  (wire (pts (xy 176.276 164.338) (xy 176.276 169.164))
+  (wire (pts (xy 173.482 164.338) (xy 173.482 169.164))
     (stroke (width 0) (type default) (color 0 0 0 0))
   )
@@
     (effects (font (size 1.27 1.27)) (justify left bottom))
   )
+  (text "Probability" (at 187.96 157.988 0)
+    (effects (font (size 2.54 2.54)) (justify left bottom))
+  )
+  (text "Noise Source" (at 103.632 88.646 0)
+    (effects (font (size 2.54 2.54)) (justify left bottom))
+  )
   (text "Tuning:\n1. Attenuate RV1 until TP_10Vpp is around 10Vpp\n2. Dial RV2 to set TP_5V to 5V\n3. Tune RV2 until OUT_OFFSET ranges from 0-10V"
     (at 82.296 69.85 0)
     (effects (font (size 1.016 1.016)) (justify left bottom))
+  )
+  (text "SNH" (at 270.764 88.138 0)
+    (effects (font (size 2.54 2.54)) (justify left bottom))
   )
   (global_label "SNH_OUTPUT" (shape input) (at 57.912 139.192 90) (fields_autoplaced)
@@
     (pin "1")
   )
-  (symbol (lib_id "Device:C") (at 176.276 172.974 180) (unit 1)
-    (in_bom yes) (on_board yes)
-    (property "Reference" "C15" (id 0) (at 170.942 172.974 90))
-    (property "Value" "100nF" (id 1) (at 172.72 172.974 90))
-    (property "Footprint" "Capacitor_SMD:C_0603_1608Metric_Pad1.08x0.95mm_HandSolder" (id 2) (at 175.3108 169.164 0)
-      (effects (font (size 1.27 1.27)) hide)
-    )
-    (property "Datasheet" "~" (id 3) (at 176.276 172.974 0)
-      (effects (font (size 1.27 1.27)) hide)
-    )
-    (property "Manufacturers Name" "YAGEO" (id 4) (at 176.276 172.974 0)
-      (effects (font (size 1.27 1.27)) hide)
-    )
-    (property "Manufacturers Part Number" "CC0805KRX7R9BB104" (id 5) (at 176.276 172.974 0)
-      (effects (font (size 1.27 1.27)) hide)
-    )
+  (symbol (lib_id "Device:C") (at 173.482 172.974 180) (unit 1)
+    (in_bom yes) (on_board yes)
+    (property "Reference" "C15" (id 0) (at 168.148 172.974 90))
+    (property "Value" "100nF" (id 1) (at 169.926 172.974 90))
+    (property "Footprint" "Capacitor_SMD:C_0603_1608Metric_Pad1.08x0.95mm_HandSolder" (id 2) (at 172.5168 169.164 0)
+      (effects (font (size 1.27 1.27)) hide)
+    )
+    (property "Datasheet" "~" (id 3) (at 173.482 172.974 0)
+      (effects (font (size 1.27 1.27)) hide)
+    )
+    (property "Manufacturers Name" "YAGEO" (id 4) (at 173.482 172.974 0)
+      (effects (font (size 1.27 1.27)) hide)
+    )
+    (property "Manufacturers Part Number" "CC0805KRX7R9BB104" (id 5) (at 173.482 172.974 0)
+      (effects (font (size 1.27 1.27)) hide)
+    )

Commit message: Updated bom with corrections in parts numbers
Parts:
- C10, C11, C12, C13, C14, C15, C16, C17, C18, C19, C8, C9: Manufacturers Part Number CC0805KRX7R9BB104 -> CC0603JRX7R9BB104
- R4, R7: Manufacturers Name (none) -> KOA Speer Electronics, Inc.; Manufacturers Part Number (none) -> RK73B1JTTD222J
Changed lines of the file:
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@@
       (effects (font (size 1.27 1.27)) hide)
     )
-    (property "Manufacturers Part Number" "CC0805KRX7R9BB104" (id 5) (at 125.984 173.99 0)
+    (property "Manufacturers Part Number" "CC0603JRX7R9BB104" (id 5) (at 125.984 173.99 0)
       (effects (font (size 1.27 1.27)) hide)
     )
@@
       (effects (font (size 1.27 1.27)) hide)
     )
-    (property "Manufacturers Part Number" "CC0805KRX7R9BB104" (id 5) (at 117.094 173.99 0)
+    (property "Manufacturers Part Number" "CC0603JRX7R9BB104" (id 5) (at 117.094 173.99 0)
       (effects (font (size 1.27 1.27)) hide)
     )
@@
       (effects (font (size 1.27 1.27)) hide)
     )
-    (property "Manufacturers Part Number" "CC0805KRX7R9BB104" (id 5) (at 108.458 184.658 0)
+    (property "Manufacturers Part Number" "CC0603JRX7R9BB104" (id 5) (at 108.458 184.658 0)
       (effects (font (size 1.27 1.27)) hide)
     )
@@
       (effects (font (size 1.27 1.27)) hide)
     )
-    (property "Manufacturers Part Number" "CC0805KRX7R9BB104" (id 5) (at 173.482 172.974 0)
+    (property "Manufacturers Part Number" "CC0603JRX7R9BB104" (id 5) (at 173.482 172.974 0)
       (effects (font (size 1.27 1.27)) hide)
     )
@@
       (effects (font (size 1.27 1.27)) hide)
     )
-    (property "Manufacturers Part Number" "CC0805KRX7R9BB104" (id 5) (at 108.458 173.99 0)
+    (property "Manufacturers Part Number" "CC0603JRX7R9BB104" (id 5) (at 108.458 173.99 0)
       (effects (font (size 1.27 1.27)) hide)
     )
@@
     )
     (property "Datasheet" "~" (id 3) (at 74.676 65.024 0)
+      (effects (font (size 1.27 1.27)) hide)
+    )
+    (property "Manufacturers Name" "KOA Speer Electronics, Inc." (id 4) (at 74.676 65.024 0)
+      (effects (font (size 1.27 1.27)) hide)
+    )
+    (property "Manufacturers Part Number" "RK73B1JTTD222J" (id 5) (at 74.676 65.024 0)
       (effects (font (size 1.27 1.27)) hide)
     )
@@
       (effects (font (size 1.27 1.27)) hide)
     )
-    (property "Manufacturers Part Number" "CC0805KRX7R9BB104" (id 5) (at 145.034 173.99 0)
+    (property "Manufacturers Part Number" "CC0603JRX7R9BB104" (id 5) (at 145.034 173.99 0)
       (effects (font (size 1.27 1.27)) hide)
     )
@@
       (effects (font (size 1.27 1.27)) hide)
     )
+    (property "Manufacturers Name" "KOA Speer Electronics, Inc." (id 4) (at 46.482 61.976 0)
+      (effects (font (size 1.27 1.27)) hide)
+    )
+    (property "Manufacturers Part Number" "RK73B1JTTD222J" (id 5) (at 46.482 61.976 0)
+      (effects (font (size 1.27 1.27)) hide)
+    )
     (pin "1")
     (pin "2")
@@
       (effects (font (size 1.27 1.27)) hide)
     )
-    (property "Manufacturers Part Number" "CC0805KRX7R9BB104" (id 5) (at 135.382 173.99 0)
+    (property "Manufacturers Part Number" "CC0603JRX7R9BB104" (id 5) (at 135.382 173.99 0)
       (effects (font (size 1.27 1.27)) hide)
     )
@@
       (effects (font (size 1.27 1.27)) hide)
     )
-    (property "Manufacturers Part Number" "CC0805KRX7R9BB104" (id 5) (at 215.9 37.592 0)
+    (property "Manufacturers Part Number" "CC0603JRX7R9BB104" (id 5) (at 215.9 37.592 0)
       (effects (font (size 1.27 1.27)) hide)
     )
@@
       (effects (font (size 1.27 1.27)) hide)
     )
-    (property "Manufacturers Part Number" "CC0805KRX7R9BB104" (id 5) (at 145.034 184.658 0)
+    (property "Manufacturers Part Number" "CC0603JRX7R9BB104" (id 5) (at 145.034 184.658 0)
       (effects (font (size 1.27 1.27)) hide)
     )
@@
       (effects (font (size 1.27 1.27)) hide)
     )
-    (property "Manufacturers Part Number" "CC0805KRX7R9BB104" (id 5) (at 135.382 184.658 0)
+    (property "Manufacturers Part Number" "CC0603JRX7R9BB104" (id 5) (at 135.382 184.658 0)
       (effects (font (size 1.27 1.27)) hide)
     )
@@
       (effects (font (size 1.27 1.27)) hide)
     )
-    (property "Manufacturers Part Number" "CC0805KRX7R9BB104" (id 5) (at 125.984 184.658 0)
+    (property "Manufacturers Part Number" "CC0603JRX7R9BB104" (id 5) (at 125.984 184.658 0)
       (effects (font (size 1.27 1.27)) hide)
     )
@@
       (effects (font (size 1.27 1.27)) hide)
     )
-    (property "Manufacturers Part Number" "CC0805KRX7R9BB104" (id 5) (at 117.094 184.658 0)
-      (effects (font (size 1.27 1.27)) hide)
-    )
+    (property "Manufacturers Part Number" "CC0603JRX7R9BB104" (id 5) (at 117.094 184.658 0)
+      (effects (font (size 1.27 1.27)) hide)
+    )

Commit message: Added footprints for 100k trimmer and 33k
Parts:
- R25: Manufacturers Name (none) -> KOA Speer; Manufacturers Part Number (none) -> CR0603-FX-3302ELF
- RV1: Manufacturers Name (none) -> Bourns; Manufacturers Part Number (none) -> PV36X104C01B00
Changed lines of the file:
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@@
+      (effects (font (size 1.27 1.27)) hide)
+    )
+    (property "Manufacturers Name" "KOA Speer" (id 4) (at 202.692 81.788 0)
+      (effects (font (size 1.27 1.27)) hide)
+    )
+    (property "Manufacturers Part Number" "CR0603-FX-3302ELF" (id 5) (at 202.692 81.788 0)
       (effects (font (size 1.27 1.27)) hide)
     )
@@
       (effects (font (size 1.27 1.27)) hide)
     )
+    (property "Manufacturers Name" "Bourns" (id 4) (at 91.186 58.928 0)
+      (effects (font (size 1.27 1.27)) hide)
+    )
+    (property "Manufacturers Part Number" "PV36X104C01B00" (id 5) (at 91.186 58.928 0)
+      (effects (font (size 1.27 1.27)) hide)
+    )
